Commit message: renamed V1 package to v1_description

File: v1_description/models/V1/urdf/V1_gazebo.urdf (robot description, URDF)
Before this commit: robot v1, 34 links, 33 joints
Links:
- removed link /v1/Head
- removed link /v1/LeftAnkleYoke
- removed link /v1/LeftElbowExtensor
- removed link /v1/LeftForearm
- removed link /v1/LeftHipAdductor
- removed link /v1/LeftHipRotator
- removed link /v1/LeftLeg
- removed link /v1/LeftPalm
- removed link /v1/LeftShankStructure
- removed link /v1/LeftShoulderAdductor
- removed link /v1/LeftShoulderExtensor
- removed link /v1/LeftShoulderRotator
- removed link /v1/LeftUpperFoot
- removed link /v1/LeftWristYoke
- removed link /v1/LowerNeckExtensor
- removed link /v1/NeckRotator
- removed link /v1/Pelvis
- removed link /v1/RightAnkleYoke
- removed link /v1/RightElbowExtensor
- removed link /v1/RightForearm
- removed link /v1/RightHipAdductor
- removed link /v1/RightHipRotator
- removed link /v1/RightLeg
- removed link /v1/RightPalm
- removed link /v1/RightShankStructure
- removed link /v1/RightShoulderAdductor
- removed link /v1/RightShoulderExtensor
- removed link /v1/RightShoulderRotator
- removed link /v1/RightUpperFoot
- removed link /v1/RightWristYoke
- removed link /v1/Trunk
- removed link /v1/WaistExtensor
- removed link /v1/WaistRotator
- removed link testbed_base
- added link v1/Head, mass 3.842; collision mesh filename=package://v1_description/models/V1/meshes/2013_05_16/head.s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; visual mesh filename=package://v1_description/models/V1/meshes/2013_05_16/head.s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
- added link v1/LeftAnkleYoke, mass 0.395; collision box size=0.033 0.076 0.025; visual box size=0.033 0.076 0.025
- added link v1/LeftElbowExtensor, mass 1.367; collision mesh filename=package://v1_description/models/V1/meshes/2013_05_16/aj4.stl; visual mesh filename=package://v1_description/models/V1/meshes/2013_05_16/aj4.stl
- added link v1/LeftForearm, mass 2.703; collision mesh filename=package://v1_description/models/V1/meshes/2013_05_16/aj5_Le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; visual mesh filename=package://v1_description/models/V1/meshes/2013_05_16/aj5_Le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
- added link v1/LeftHipAdductor, mass 5.15; collision mesh filename=package://v1_description/models/V1/meshes/2013_05_16/lj2.stl; visual mesh filename=package://v1_description/models/V1/meshes/2013_05_16/lj2.stl
- added link v1/LeftHipRotator, mass 2.39; collision mesh filename=package://v1_description/models/V1/meshes/2013_05_16/lj1_Le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; visual mesh filename=package://v1_description/models/V1/meshes/2013_05_16/lj1_Le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
- added link v1/LeftLeg, mass 7.14; collision mesh filename=package://v1_description/models/V1/meshes/2013_05_16/lj3_Le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; visual mesh filename=package://v1_description/models/V1/meshes/2013_05_16/lj3_Le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
- added link v1/LeftPalm, mass 0.712; collision mesh filename=package://v1_description/models/V1/meshes/2013_05_16/palm_L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; visual mesh filename=package://v1_description/models/V1/meshes/2013_05_16/palm_L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
- added link v1/LeftShankStructure, mass 6.902; collision mesh filename=package://v1_description/models/V1/meshes/2013_05_16/lj4_Le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; visual mesh filename=package://v1_description/models/V1/meshes/2013_05_16/lj4_Le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
- added link v1/LeftShoulderAdductor, mass 3.67; collision mesh filename=package://v1_description/models/V1/meshes/2013_05_16/aj2.stl; visual mesh filename=package://v1_description/models/V1/meshes/2013_05_16/aj2.stl
- added link v1/LeftShoulderExtensor, mass 2.45; collision mesh filename=package://v1_description/models/V1/meshes/2013_05_16/aj1_Le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; visual mesh filename=package://v1_description/models/V1/meshes/2013_05_16/aj1_Le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
- added link v1/LeftShoulderRotator, mass 2.575; collision mesh filename=package://v1_description/models/V1/meshes/2013_05_16/aj3_Le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; visual mesh filename=package://v1_description/models/V1/meshes/2013_05_16/aj3_Le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
- added link v1/LeftUpperFoot, mass 1.888; collision box size=0.082 0.128 0.3; visual mesh filename=package://v1_description/models/V1/meshes/2013_05_16/lj6_Le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
- added link v1/LeftWristYoke, mass 0.1; collision box size=0.03 0.01 0.051; visual box size=0.03 0.01 0.051
- added link v1/LowerNeckExtensor, mass 0.1; collision mesh filename=package://v1_description/models/V1/meshes/2013_05_16/nj1.stl; visual mesh filename=package://v1_description/models/V1/meshes/2013_05_16/nj1.stl
- added link v1/NeckRotator, mass 0.1; collision mesh filename=package://v1_description/models/V1/meshes/2013_05_16/nj2.stl; visual mesh filename=package://v1_description/models/V1/meshes/2013_05_16/nj2.stl
- added link v1/Pelvis, mass 5.15; collision mesh filename=package://v1_description/models/V1/meshes/2013_05_16/pelvis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; visual mesh filename=package://v1_description/models/V1/meshes/2013_05_16/pelvis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
- added link v1/RightAnkleYoke, mass 0.395; collision box size=0.033 0.076 0.025; visual box size=0.033 0.076 0.025
- added link v1/RightElbowExtensor, mass 1.367; collision mesh filename=package://v1_description/models/V1/meshes/2013_05_16/aj4.stl; visual mesh filename=package://v1_description/models/V1/meshes/2013_05_16/aj4.stl
- added link v1/RightForearm, mass 2.703; collision mesh filename=package://v1_description/models/V1/meshes/2013_05_16/aj5_Ri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; visual mesh filename=package://v1_description/models/V1/meshes/2013_05_16/aj5_Ri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
- added link v1/RightHipAdductor, mass 5.15; collision mesh filename=package://v1_description/models/V1/meshes/2013_05_16/lj2.stl; visual mesh filename=package://v1_description/models/V1/meshes/2013_05_16/lj2.stl
- added link v1/RightHipRotator, mass 2.39; collision mesh filename=package://v1_description/models/V1/meshes/2013_05_16/lj1_Ri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; visual mesh filename=package://v1_description/models/V1/meshes/2013_05_16/lj1_Ri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
- added link v1/RightLeg, mass 7.14; collision mesh filename=package://v1_description/models/V1/meshes/2013_05_16/lj3_Ri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; visual mesh filename=package://v1_description/models/V1/meshes/2013_05_16/lj3_Ri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
- added link v1/RightPalm, mass 0.712; collision mesh filename=package://v1_description/models/V1/meshes/2013_05_16/palm_R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; visual mesh filename=package://v1_description/models/V1/meshes/2013_05_16/palm_R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
- added link v1/RightShankStructure, mass 6.902; collision mesh filename=package://v1_description/models/V1/meshes/2013_05_16/lj4_Ri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; visual mesh filename=package://v1_description/models/V1/meshes/2013_05_16/lj4_Ri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
- added link v1/RightShoulderAdductor, mass 3.67; collision mesh filename=package://v1_description/models/V1/meshes/2013_05_16/aj2.stl; visual mesh filename=package://v1_description/models/V1/meshes/2013_05_16/aj2.stl
- added link v1/RightShoulderExtensor, mass 2.45; collision mesh filename=package://v1_description/models/V1/meshes/2013_05_16/aj1_Ri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; visual mesh filename=package://v1_description/models/V1/meshes/2013_05_16/aj1_Ri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
- added link v1/RightShoulderRotator, mass 2.575; collision mesh filename=package://v1_description/models/V1/meshes/2013_05_16/aj3_Ri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; visual mesh filename=package://v1_description/models/V1/meshes/2013_05_16/aj3_Ri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
- added link v1/RightUpperFoot, mass 1.888; collision box size=0.082 0.128 0.3; visual mesh filename=package://v1_description/models/V1/meshes/2013_05_16/lj6_Ri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
- added link v1/RightWristYoke, mass 0.1; collision box size=0.03 0.01 0.051; visual box size=0.03 0.01 0.051
- added link v1/Trunk, mass 38.3; collision mesh filename=package://v1_description/models/V1/meshes/2013_05_16/wj3.stl; visual mesh filename=package://v1_description/models/V1/meshes/2013_05_16/wj3.stl
- added link v1/WaistExtensor, mass 0.1
- added link v1/WaistRotator, mass 0.1
- added link world, mass 0.1
Joints:
- joint LeftAnkle: child /v1/LeftUpperFoot -> v1/LeftUpperFoot; parent /v1/LeftAnkleYoke -> v1/LeftAnkleYoke
- joint LeftAnkleExtensor: child /v1/LeftAnkleYoke -> v1/LeftAnkleYoke; parent /v1/LeftShankStructure -> v1/LeftShankStructure
- joint LeftElbowExtensor: child /v1/LeftElbowExtensor -> v1/LeftElbowExtensor; parent /v1/LeftShoulderRotator -> v1/LeftShoulderRotator
- joint LeftForearmSupinator: child /v1/LeftForearm -> v1/LeftForearm; parent /v1/LeftElbowExtensor -> v1/LeftElbowExtensor
- joint LeftHipAdductor: child /v1/LeftHipAdductor -> v1/LeftHipAdductor; parent /v1/LeftHipRotator -> v1/LeftHipRotator
- joint LeftHipExtensor: child /v1/LeftLeg -> v1/LeftLeg; parent /v1/LeftHipAdductor -> v1/LeftHipAdductor
- joint LeftHipRotator: child /v1/LeftHipRotator -> v1/LeftHipRotator; parent /v1/Pelvis -> v1/Pelvis
- joint LeftKneeExtensor: child /v1/LeftShankStructure -> v1/LeftShankStructure; parent /v1/LeftLeg -> v1/LeftLeg
- joint LeftShoulderAdductor: child /v1/LeftShoulderAdductor -> v1/LeftShoulderAdductor; parent /v1/LeftShoulderExtensor -> v1/LeftShoulderExtensor
- joint LeftShoulderExtensor: child /v1/LeftShoulderExtensor -> v1/LeftShoulderExtensor; parent /v1/Trunk -> v1/Trunk
- joint LeftShoulderSupinator: child /v1/LeftShoulderRotator -> v1/LeftShoulderRotator; parent /v1/LeftShoulderAdductor -> v1/LeftShoulderAdductor
- joint LeftWrist: child /v1/LeftPalm -> v1/LeftPalm; parent /v1/LeftWristYoke -> v1/LeftWristYoke
- joint LeftWristExtensor: child /v1/LeftWristYoke -> v1/LeftWristYoke; parent /v1/LeftForearm -> v1/LeftForearm
- joint LowerNeckExtensor: child /v1/LowerNeckExtensor -> v1/LowerNeckExtensor; parent /v1/Trunk -> v1/Trunk
- joint NeckRotator: child /v1/NeckRotator -> v1/NeckRotator; parent /v1/LowerNeckExtensor -> v1/LowerNeckExtensor
- joint RightAnkle: child /v1/RightUpperFoot -> v1/RightUpperFoot; parent /v1/RightAnkleYoke -> v1/RightAnkleYoke
- joint RightAnkleExtensor: child /v1/RightAnkleYoke -> v1/RightAnkleYoke; parent /v1/RightShankStructure -> v1/RightShankStructure
- joint RightElbowExtensor: child /v1/RightElbowExtensor -> v1/RightElbowExtensor; parent /v1/RightShoulderRotator -> v1/RightShoulderRotator
- joint RightForearmSupinator: child /v1/RightForearm -> v1/RightForearm; parent /v1/RightElbowExtensor -> v1/RightElbowExtensor
- joint RightHipAdductor: child /v1/RightHipAdductor -> v1/RightHipAdductor; parent /v1/RightHipRotator -> v1/RightHipRotator
- joint RightHipExtensor: child /v1/RightLeg -> v1/RightLeg; parent /v1/RightHipAdductor -> v1/RightHipAdductor
- joint RightHipRotator: child /v1/RightHipRotator -> v1/RightHipRotator; parent /v1/Pelvis -> v1/Pelvis
- joint RightKneeExtensor: child /v1/RightShankStructure -> v1/RightShankStructure; parent /v1/RightLeg -> v1/RightLeg
- joint RightShoulderAdductor: child /v1/RightShoulderAdductor -> v1/RightShoulderAdductor; parent /v1/RightShoulderExtensor -> v1/RightShoulderExtensor
- joint RightShoulderExtensor: child /v1/RightShoulderExtensor -> v1/RightShoulderExtensor; parent /v1/Trunk -> v1/Trunk
- joint RightShoulderSupinator: child /v1/RightShoulderRotator -> v1/RightShoulderRotator; parent /v1/RightShoulderAdductor -> v1/RightShoulderAdductor
- joint RightWrist: child /v1/RightPalm -> v1/RightPalm; parent /v1/RightWristYoke -> v1/RightWristYoke
- joint RightWristExtensor: child /v1/RightWristYoke -> v1/RightWristYoke; parent /v1/RightForearm -> v1/RightForearm
- joint UpperNeckExtensor: child /v1/Head -> v1/Head; parent /v1/NeckRotator -> v1/NeckRotator
- joint WaistExtensor: child /v1/WaistExtensor -> v1/WaistExtensor; parent /v1/WaistRotator -> v1/WaistRotator
- joint WaistLateralExtensor: child /v1/Trunk -> v1/Trunk; parent /v1/WaistExtensor -> v1/WaistExtensor
- joint WaistRotator: child /v1/WaistRotator -> v1/WaistRotator; parent /v1/Pelvis -> v1/Pelvis
- joint pelvisOffset: child /v1/Pelvis -> v1/Pelvis; origin xyz=0 0 0.0 rpy=0 0 0 -> xyz=0 0 1.2 rpy=0 -0.2 0; parent testbed_base -> world

File: v1_description/models/V1/xacro/arm/arm.xacro (robot description, xacro)
@@ -5,10 +5,10 @@
             http://bender.jsc.nasa.gov/confluence/pages/viewpage.action?pageId=16417593
   -->
-  <xacro:include filename="$(find V1)/models/V1/xacro/arm/joint_names.xacro"/>
-  <xacro:include filename="$(find V1)/models/V1/xacro/arm/link_names.xacro"/>
-  <xacro:include filename="$(find V1)/models/V1/xacro/arm/joint_limits.xacro"/>
-  <xacro:include filename="$(find V1)/models/V1/xacro/arm/dh_parameters.xacro"/>
-  <xacro:include filename="$(find V1)/models/V1/xacro/arm/mass_parameters.xacro"/>
-  <xacro:include filename="$(find V1)/models/V1/xacro/sensors/camboard.xacro"/>
+  <xacro:include filename="$(find v1_description)/models/V1/xacro/arm/joint_names.xacro"/>
+  <xacro:include filename="$(find v1_description)/models/V1/xacro/arm/link_names.xacro"/>
+  <xacro:include filename="$(find v1_description)/models/V1/xacro/arm/joint_limits.xacro"/>
+  <xacro:include filename="$(find v1_description)/models/V1/xacro/arm/dh_parameters.xacro"/>
+  <xacro:include filename="$(find v1_description)/models/V1/xacro/arm/mass_parameters.xacro"/>
+  <xacro:include filename="$(find v1_description)/models/V1/xacro/sensors/camboard.xacro"/>
   <!-- Link properties. -->
   <!-- <xacro:property name="AJ1_Link_Radius" value="0.080" />

File: v1_description/models/V1/xacro/head/head.xacro (robot description, xacro)
@@ -5,14 +5,14 @@
   -->
   <!-- Properties -->
-  <xacro:include filename="$(find V1)/models/V1/xacro/head/joint_names.xacro"/>
-  <xacro:include filename="$(find V1)/models/V1/xacro/head/link_names.xacro"/>
-  <xacro:include filename="$(find V1)/models/V1/xacro/head/joint_limits.xacro"/>
-  <xacro:include filename="$(find V1)/models/V1/xacro/head/dh_parameters.xacro"/>
-  <xacro:include filename="$(find V1)/models/V1/xacro/head/mass_parameters.xacro"/>
-  <xacro:include filename="$(find V1)/models/V1/xacro/sensors/camboard.xacro"/>
-  <xacro:include filename="$(find V1)/models/V1/xacro/sensors/flea.xacro"/>
-  <xacro:include filename="$(find V1)/models/V1/xacro/sensors/ibeo.xacro"/>
-  <!-- <xacro:include filename="$(find V1)/models/V1/xacro/sensors/asus.xacro"/> -->
-  <xacro:include filename="$(find V1)/models/V1/xacro/sensors/ensenso.xacro"/>
+  <xacro:include filename="$(find v1_description)/models/V1/xacro/head/joint_names.xacro"/>
+  <xacro:include filename="$(find v1_description)/models/V1/xacro/head/link_names.xacro"/>
+  <xacro:include filename="$(find v1_description)/models/V1/xacro/head/joint_limits.xacro"/>
+  <xacro:include filename="$(find v1_description)/models/V1/xacro/head/dh_parameters.xacro"/>
+  <xacro:include filename="$(find v1_description)/models/V1/xacro/head/mass_parameters.xacro"/>
+  <xacro:include filename="$(find v1_description)/models/V1/xacro/sensors/camboard.xacro"/>
+  <xacro:include filename="$(find v1_description)/models/V1/xacro/sensors/flea.xacro"/>
+  <xacro:include filename="$(find v1_description)/models/V1/xacro/sensors/ibeo.xacro"/>
+  <!-- <xacro:include filename="$(find v1_description)/models/V1/xacro/sensors/asus.xacro"/> -->
+  <xacro:include filename="$(find v1_description)/models/V1/xacro/sensors/ensenso.xacro"/>
   <!-- Link properties. -->
   <xacro:property name="NJ3_Link_Radius" value="0.14"/>

File: v1_description/models/V1/xacro/leg/leg.xacro (robot description, xacro)
@@ -5,12 +5,12 @@
             http://bender.jsc.nasa.gov/confluence/pages/viewpage.action?pageId=16417593
   -->
-  <xacro:include filename="$(find V1)/models/V1/xacro/leg/joint_names.xacro"/>
-  <xacro:include filename="$(find V1)/models/V1/xacro/leg/link_names.xacro"/>
-  <xacro:include filename="$(find V1)/models/V1/xacro/leg/joint_limits.xacro"/>
-  <xacro:include filename="$(find V1)/models/V1/xacro/leg/dh_parameters.xacro"/>
-  <xacro:include filename="$(find V1)/models/V1/xacro/leg/mass_parameters.xacro"/>
-  <xacro:include filename="$(find V1)/models/V1/xacro/sensors/camboard.xacro"/>
-  <xacro:include filename="$(find V1)/models/V1/xacro/sensors/hokuyo.xacro"/>
-  <xacro:include filename="$(find V1)/models/V1/xacro/sensors/hw_sensors.xacro"/>
+  <xacro:include filename="$(find v1_description)/models/V1/xacro/leg/joint_names.xacro"/>
+  <xacro:include filename="$(find v1_description)/models/V1/xacro/leg/link_names.xacro"/>
+  <xacro:include filename="$(find v1_description)/models/V1/xacro/leg/joint_limits.xacro"/>
+  <xacro:include filename="$(find v1_description)/models/V1/xacro/leg/dh_parameters.xacro"/>
+  <xacro:include filename="$(find v1_description)/models/V1/xacro/leg/mass_parameters.xacro"/>
+  <xacro:include filename="$(find v1_description)/models/V1/xacro/sensors/camboard.xacro"/>
+  <xacro:include filename="$(find v1_description)/models/V1/xacro/sensors/hokuyo.xacro"/>
+  <xacro:include filename="$(find v1_description)/models/V1/xacro/sensors/hw_sensors.xacro"/>
   <!-- Link properties. -->
   <xacro:property name="LJ1_Link_Width" value="0.149"/>

File: v1_description/models/V1/xacro/little_finger/little_finger.xacro (robot description, xacro)
@@ -5,10 +5,10 @@
             http://bender.jsc.nasa.gov/confluence/pages/viewpage.action?pageId=16417593
   -->
-  <xacro:include filename="$(find V1)/models/V1/xacro/little_finger/joint_names.xacro"/>
-  <xacro:include filename="$(find V1)/models/V1/xacro/little_finger/actuator_names.xacro"/>
-  <xacro:include filename="$(find V1)/models/V1/xacro/little_finger/link_names.xacro"/>
-  <xacro:include filename="$(find V1)/models/V1/xacro/little_finger/joint_limits.xacro"/>
-  <xacro:include filename="$(find V1)/models/V1/xacro/little_finger/dh_parameters.xacro"/>
-  <xacro:include filename="$(find V1)/models/V1/xacro/little_finger/mass_parameters.xacro"/>
+  <xacro:include filename="$(find v1_description)/models/V1/xacro/little_finger/joint_names.xacro"/>
+  <xacro:include filename="$(find v1_description)/models/V1/xacro/little_finger/actuator_names.xacro"/>
+  <xacro:include filename="$(find v1_description)/models/V1/xacro/little_finger/link_names.xacro"/>
+  <xacro:include filename="$(find v1_description)/models/V1/xacro/little_finger/joint_limits.xacro"/>
+  <xacro:include filename="$(find v1_description)/models/V1/xacro/little_finger/dh_parameters.xacro"/>
+  <xacro:include filename="$(find v1_description)/models/V1/xacro/little_finger/mass_parameters.xacro"/>
   <!-- Link properties. -->
   <xacro:property name="LFJ1_Link_Width" value="0.010"/>

File: v1_description/models/V1/xacro/middle_finger/middle_finger.xacro (robot description, xacro)
@@ -5,10 +5,10 @@
             http://bender.jsc.nasa.gov/confluence/pages/viewpage.action?pageId=16417593
   -->
-  <xacro:include filename="$(find V1)/models/V1/xacro/middle_finger/joint_names.xacro"/>
-  <xacro:include filename="$(find V1)/models/V1/xacro/middle_finger/actuator_names.xacro"/>
-  <xacro:include filename="$(find V1)/models/V1/xacro/middle_finger/link_names.xacro"/>
-  <xacro:include filename="$(find V1)/models/V1/xacro/middle_finger/joint_limits.xacro"/>
-  <xacro:include filename="$(find V1)/models/V1/xacro/middle_finger/dh_parameters.xacro"/>
-  <xacro:include filename="$(find V1)/models/V1/xacro/middle_finger/mass_parameters.xacro"/>
+  <xacro:include filename="$(find v1_description)/models/V1/xacro/middle_finger/joint_names.xacro"/>
+  <xacro:include filename="$(find v1_description)/models/V1/xacro/middle_finger/actuator_names.xacro"/>
+  <xacro:include filename="$(find v1_description)/models/V1/xacro/middle_finger/link_names.xacro"/>
+  <xacro:include filename="$(find v1_description)/models/V1/xacro/middle_finger/joint_limits.xacro"/>
+  <xacro:include filename="$(find v1_description)/models/V1/xacro/middle_finger/dh_parameters.xacro"/>
+  <xacro:include filename="$(find v1_description)/models/V1/xacro/middle_finger/mass_parameters.xacro"/>
   <!-- Link properties. -->
   <xacro:property name="MFJ1_Link_Width" value="0.054"/>

File: v1_description/models/V1/xacro/primary_finger/primary_finger.xacro (robot description, xacro)
@@ -5,10 +5,10 @@
             http://bender.jsc.nasa.gov/confluence/pages/viewpage.action?pageId=16417593
   -->
-  <xacro:include filename="$(find V1)/models/V1/xacro/primary_finger/joint_names.xacro"/>
-  <xacro:include filename="$(find V1)/models/V1/xacro/primary_finger/actuator_names.xacro"/>
-  <xacro:include filename="$(find V1)/models/V1/xacro/primary_finger/link_names.xacro"/>
-  <xacro:include filename="$(find V1)/models/V1/xacro/primary_finger/joint_limits.xacro"/>
-  <xacro:include filename="$(find V1)/models/V1/xacro/primary_finger/dh_parameters.xacro"/>
-  <xacro:include filename="$(find V1)/models/V1/xacro/primary_finger/mass_parameters.xacro"/>
+  <xacro:include filename="$(find v1_description)/models/V1/xacro/primary_finger/joint_names.xacro"/>
+  <xacro:include filename="$(find v1_description)/models/V1/xacro/primary_finger/actuator_names.xacro"/>
+  <xacro:include filename="$(find v1_description)/models/V1/xacro/primary_finger/link_names.xacro"/>
+  <xacro:include filename="$(find v1_description)/models/V1/xacro/primary_finger/joint_limits.xacro"/>
+  <xacro:include filename="$(find v1_description)/models/V1/xacro/primary_finger/dh_parameters.xacro"/>
+  <xacro:include filename="$(find v1_description)/models/V1/xacro/primary_finger/mass_parameters.xacro"/>
   <!-- Link properties. -->
   <xacro:property name="PFJ1_Link_Width" value="0.029"/>

File: v1_description/models/V1/xacro/thumb/thumb.xacro (robot description, xacro)
@@ -5,10 +5,10 @@
             http://bender.jsc.nasa.gov/confluence/pages/viewpage.action?pageId=16417593
   -->
-  <xacro:include filename="$(find V1)/models/V1/xacro/thumb/joint_names.xacro"/>
-  <xacro:include filename="$(find V1)/models/V1/xacro/thumb/actuator_names.xacro"/>
-  <xacro:include filename="$(find V1)/models/V1/xacro/thumb/link_names.xacro"/>
-  <xacro:include filename="$(find V1)/models/V1/xacro/thumb/joint_limits.xacro"/>
-  <xacro:include filename="$(find V1)/models/V1/xacro/thumb/dh_parameters.xacro"/>
-  <xacro:include filename="$(find V1)/models/V1/xacro/thumb/mass_parameters.xacro"/>
+  <xacro:include filename="$(find v1_description)/models/V1/xacro/thumb/joint_names.xacro"/>
+  <xacro:include filename="$(find v1_description)/models/V1/xacro/thumb/actuator_names.xacro"/>
+  <xacro:include filename="$(find v1_description)/models/V1/xacro/thumb/link_names.xacro"/>
+  <xacro:include filename="$(find v1_description)/models/V1/xacro/thumb/joint_limits.xacro"/>
+  <xacro:include filename="$(find v1_description)/models/V1/xacro/thumb/dh_parameters.xacro"/>
+  <xacro:include filename="$(find v1_description)/models/V1/xacro/thumb/mass_parameters.xacro"/>
   <!-- Link properties. -->
   <xacro:property name="TJ1_Link_Width" value="0.010"/>

File: v1_description/models/V1/xacro/v1.xacro (robot description, xacro)
@@ -4,6 +4,6 @@
 			xmlns:sensor="http://playerstage.sourceforge.net/gazebo/xmlschema/#sensor"
 			xmlns:xacro="http://playerstage.sourceforge.net/gazebo/xmlschema/#interface">
-  <xacro:property name="mesh_root" value="package://V1/models/V1/meshes/2013_05_16"/>
+  <xacro:property name="mesh_root" value="package://v1_description/models/V1/meshes/2013_05_16"/>
   <xacro:property name="robot_name" value= "v1/"/>
-  <xacro:include filename="$(find V1)/models/V1/xacro/V1_sim_base.xacro"/>
+  <xacro:include filename="$(find v1_description)/models/V1/xacro/V1_sim_base.xacro"/>
 </robot>
