Commit message: renamed V1 package to v1_description

File: v1_description/models/V1/xacro/waist/waist.xacro (robot description, xacro)
@@ -5,12 +5,12 @@
   -->
   <!-- Properties -->
-  <xacro:include filename="$(find V1)/models/V1/xacro/waist/joint_names.xacro"/>
-  <xacro:include filename="$(find V1)/models/V1/xacro/waist/link_names.xacro"/>
-  <xacro:include filename="$(find V1)/models/V1/xacro/waist/joint_limits.xacro"/>
-  <xacro:include filename="$(find V1)/models/V1/xacro/waist/dh_parameters.xacro"/>
-  <xacro:include filename="$(find V1)/models/V1/xacro/waist/mass_parameters.xacro"/>
-  <xacro:include filename="$(find V1)/models/V1/xacro/sensors/microstrain.xacro"/>
-  <xacro:include filename="$(find V1)/models/V1/xacro/sensors/virtual_sensor.xacro"/>
-  <xacro:include filename="$(find V1)/models/V1/xacro/sensors/flea.xacro"/>
+  <xacro:include filename="$(find v1_description)/models/V1/xacro/waist/joint_names.xacro"/>
+  <xacro:include filename="$(find v1_description)/models/V1/xacro/waist/link_names.xacro"/>
+  <xacro:include filename="$(find v1_description)/models/V1/xacro/waist/joint_limits.xacro"/>
+  <xacro:include filename="$(find v1_description)/models/V1/xacro/waist/dh_parameters.xacro"/>
+  <xacro:include filename="$(find v1_description)/models/V1/xacro/waist/mass_parameters.xacro"/>
+  <xacro:include filename="$(find v1_description)/models/V1/xacro/sensors/microstrain.xacro"/>
+  <xacro:include filename="$(find v1_description)/models/V1/xacro/sensors/virtual_sensor.xacro"/>
+  <xacro:include filename="$(find v1_description)/models/V1/xacro/sensors/flea.xacro"/>
   <!-- TODO: Get waist approximation correct -->
   <xacro:property name="Trunk_Width" value="0.477"/>

File: v1_gazebo/models/urdf/V1_gazebo.urdf (robot description, URDF)
Before this commit: robot v1, 34 links, 33 joints
Links:
- link v1/Head: geometry collision mesh filename=package://v1_description/models/V1/meshes/2013_05_16/head.s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; visual mesh filename=package://v1_description/models/V1/meshes/2013_05_16/head.s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
- link v1/LeftElbowExtensor: geometry collision mesh filename=package://v1_description/models/V1/meshes/2013_05_16/aj4.stl; visual mesh filename=package://v1_description/models/V1/meshes/2013_05_16/aj4.stl
- link v1/LeftForearm: geometry collision mesh filename=package://v1_description/models/V1/meshes/2013_05_16/aj5_Le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; visual mesh filename=package://v1_description/models/V1/meshes/2013_05_16/aj5_Le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
- link v1/LeftHipAdductor: geometry collision mesh filename=package://v1_description/models/V1/meshes/2013_05_16/lj2.stl; visual mesh filename=package://v1_description/models/V1/meshes/2013_05_16/lj2.stl
- link v1/LeftHipRotator: geometry collision mesh filename=package://v1_description/models/V1/meshes/2013_05_16/lj1_Le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; visual mesh filename=package://v1_description/models/V1/meshes/2013_05_16/lj1_Le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
- link v1/LeftLeg: geometry collision mesh filename=package://v1_description/models/V1/meshes/2013_05_16/lj3_Le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; visual mesh filename=package://v1_description/models/V1/meshes/2013_05_16/lj3_Le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
- link v1/LeftPalm: geometry collision mesh filename=package://v1_description/models/V1/meshes/2013_05_16/palm_L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; visual mesh filename=package://v1_description/models/V1/meshes/2013_05_16/palm_L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
- link v1/LeftShankStructure: geometry collision mesh filename=package://v1_description/models/V1/meshes/2013_05_16/lj4_Le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; visual mesh filename=package://v1_description/models/V1/meshes/2013_05_16/lj4_Le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
- link v1/LeftShoulderAdductor: geometry collision mesh filename=package://v1_description/models/V1/meshes/2013_05_16/aj2.stl; visual mesh filename=package://v1_description/models/V1/meshes/2013_05_16/aj2.stl
- link v1/LeftShoulderExtensor: geometry collision mesh filename=package://v1_description/models/V1/meshes/2013_05_16/aj1_Le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; visual mesh filename=package://v1_description/models/V1/meshes/2013_05_16/aj1_Le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
- link v1/LeftShoulderRotator: geometry collision mesh filename=package://v1_description/models/V1/meshes/2013_05_16/aj3_Le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; visual mesh filename=package://v1_description/models/V1/meshes/2013_05_16/aj3_Le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
- link v1/LeftUpperFoot: geometry collision box size=0.082 0.128 0.3; visual mesh filename=package://v1_description/models/V1/meshes/2013_05_16/lj6_Le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
- link v1/LowerNeckExtensor: geometry collision mesh filename=package://v1_description/models/V1/meshes/2013_05_16/nj1.stl; visual mesh filename=package://v1_description/models/V1/meshes/2013_05_16/nj1.stl
- link v1/NeckRotator: geometry collision mesh filename=package://v1_description/models/V1/meshes/2013_05_16/nj2.stl; visual mesh filename=package://v1_description/models/V1/meshes/2013_05_16/nj2.stl
- link v1/Pelvis: geometry collision mesh filename=package://v1_description/models/V1/meshes/2013_05_16/pelvis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; visual mesh filename=package://v1_description/models/V1/meshes/2013_05_16/pelvis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
- link v1/RightElbowExtensor: geometry collision mesh filename=package://v1_description/models/V1/meshes/2013_05_16/aj4.stl; visual mesh filename=package://v1_description/models/V1/meshes/2013_05_16/aj4.stl
- link v1/RightForearm: geometry collision mesh filename=package://v1_description/models/V1/meshes/2013_05_16/aj5_Ri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; visual mesh filename=package://v1_description/models/V1/meshes/2013_05_16/aj5_Ri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
- link v1/RightHipAdductor: geometry collision mesh filename=package://v1_description/models/V1/meshes/2013_05_16/lj2.stl; visual mesh filename=package://v1_description/models/V1/meshes/2013_05_16/lj2.stl
- link v1/RightHipRotator: geometry collision mesh filename=package://v1_description/models/V1/meshes/2013_05_16/lj1_Ri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; visual mesh filename=package://v1_description/models/V1/meshes/2013_05_16/lj1_Ri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
- link v1/RightLeg: geometry collision mesh filename=package://v1_description/models/V1/meshes/2013_05_16/lj3_Ri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; visual mesh filename=package://v1_description/models/V1/meshes/2013_05_16/lj3_Ri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
- link v1/RightPalm: geometry collision mesh filename=package://v1_description/models/V1/meshes/2013_05_16/palm_R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; visual mesh filename=package://v1_description/models/V1/meshes/2013_05_16/palm_R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
- link v1/RightShankStructure: geometry collision mesh filename=package://v1_description/models/V1/meshes/2013_05_16/lj4_Ri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; visual mesh filename=package://v1_description/models/V1/meshes/2013_05_16/lj4_Ri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
- link v1/RightShoulderAdductor: geometry collision mesh filename=package://v1_description/models/V1/meshes/2013_05_16/aj2.stl; visual mesh filename=package://v1_description/models/V1/meshes/2013_05_16/aj2.stl
- link v1/RightShoulderExtensor: geometry collision mesh filename=package://v1_description/models/V1/meshes/2013_05_16/aj1_Ri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; visual mesh filename=package://v1_description/models/V1/meshes/2013_05_16/aj1_Ri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
- link v1/RightShoulderRotator: geometry collision mesh filename=package://v1_description/models/V1/meshes/2013_05_16/aj3_Ri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; visual mesh filename=package://v1_description/models/V1/meshes/2013_05_16/aj3_Ri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
- link v1/RightUpperFoot: geometry collision box size=0.082 0.128 0.3; visual mesh filename=package://v1_description/models/V1/meshes/2013_05_16/lj6_Ri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
- link v1/Trunk: geometry collision mesh filename=package://v1_description/models/V1/meshes/2013_05_16/wj3.stl; visual mesh filename=package://v1_description/models/V1/meshes/2013_05_16/wj3.stl

File: v1_gazebo/models/xacro/v1_gazebo.xacro (robot description, xacro)
@@ -4,5 +4,5 @@
 			xmlns:sensor="http://playerstage.sourceforge.net/gazebo/xmlschema/#sensor"
 			xmlns:xacro="http://playerstage.sourceforge.net/gazebo/xmlschema/#interface">
-  <xacro:property name="mesh_root" value="package://V1/models/V1/meshes/2013_05_16"/>
+  <xacro:property name="mesh_root" value="package://v1_description/models/V1/meshes/2013_05_16"/>
   <xacro:property name="robot_name" value= "v1/"/>
   <xacro:include filename="$(find v1_gazebo)/models/xacro/v1_sim_base.xacro"/>

File: v1_gazebo/models/xacro/v1_sim_base.xacro (robot description, xacro)
@@ -8,7 +8,7 @@
     <xacro:include filename="$(find common_xacro)/xacro/common_properties.xacro" />
     <xacro:include filename="$(find common_xacro)/xacro/materials.xacro" />
-    <xacro:include filename="$(find V1)/models/V1/xacro/common/common_bodies.xacro" />
-    <xacro:include filename="$(find V1)/models/V1/xacro/utility/utility.xacro" />
-    <xacro:include filename="$(find V1)/models/V1/xacro/common/actuator_names.xacro" />
+    <xacro:include filename="$(find v1_description)/models/V1/xacro/common/common_bodies.xacro" />
+    <xacro:include filename="$(find v1_description)/models/V1/xacro/utility/utility.xacro" />
+    <xacro:include filename="$(find v1_description)/models/V1/xacro/common/actuator_names.xacro" />
     <!-- ===== DUMMY 'BASE' LINK ==== -->
     <xacro:virtual_link name="world"
@@ -20,8 +20,8 @@
                        origin_rpy="0 -0.2 0" />
      <!-- ===== PUBLISH ODOMETRY DATA ==== -->
-    <xacro:include filename="$(find V1)/models/V1/xacro/sensors/pos3d.xacro" />
+    <xacro:include filename="$(find v1_description)/models/V1/xacro/sensors/pos3d.xacro" />
     <xacro:v1_absolute_pose parentLink="v1/Trunk" topicName="v1/pose" origin_xyz="0 0 0" origin_rpy="0 0 0"/>
     <!-- ===== PUBLISH ODOMETRY DATA ==== -->
-    <xacro:include filename="$(find V1)/models/V1/xacro/sensors/pos3d.xacro" />
+    <xacro:include filename="$(find v1_description)/models/V1/xacro/sensors/pos3d.xacro" />
     <xacro:v1_absolute_pose parentLink="v1/Pelvis" topicName="v1/Pelvis/pose" origin_xyz="0 0 0" origin_rpy="0 0 0"/>
     <!-- ===== PELVIS ===== -->
